File: ft2232.kicad_sch (KiCad schematic)
At the start: 30 parts, among them U2 FT2232HL

Commit message: erc ok
Parts:
- gave numbers to parts that had none: 29

Commit message: wip footprint assoc
Parts:
- C10, C11, C6: value 10uF -> 10uF/25V; footprint (none) -> Capacitor_SMD:C_1206_3216Metric
- C12, C13, C14, C15, C16, C17, C18, C19, C5, C7: value 100nF -> 100nF/50V; footprint (none) -> Capacitor_SMD:C_0603_1608Metric
- C8, C9: footprint (none) -> Capacitor_SMD:C_0603_1608Metric
- D3, D4: footprint (none) -> LED_SMD:LED_0603_1608Metric
Changed lines of the file:
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@@
   (symbol (lib_id "power:PWR_FLAG") (at 106.68 24.13 0) (unit 1)
     (in_bom yes) (on_board yes)
-    (property "Reference" "#FLG?" (id 0) (at 106.68 22.225 0)
+    (property "Reference" "#FLG04" (id 0) (at 106.68 22.225 0)
       (effects (font (size 1.27 1.27)) hide)
     )
@@
     (property "Reference" "D3" (id 0) (at 201.93 113.03 0))
     (property "Value" "LED" (id 1) (at 201.93 115.57 0))
-    (property "Footprint" "" (id 2) (at 201.93 118.11 0)
+    (property "Footprint" "LED_SMD:LED_0603_1608Metric" (id 2) (at 201.93 118.11 0)
       (effects (font (size 1.27 1.27)) hide)
     )
@@
     (property "Reference" "D4" (id 0) (at 201.93 121.92 0))
     (property "Value" "LED" (id 1) (at 201.93 124.46 0))
-    (property "Footprint" "" (id 2) (at 201.93 127 0)
+    (property "Footprint" "LED_SMD:LED_0603_1608Metric" (id 2) (at 201.93 127 0)
       (effects (font (size 1.27 1.27)) hide)
     )
@@
       (effects (font (size 1.27 1.27)) (justify left))
     )
-    (property "Value" "100nF" (id 1) (at 55.88 92.71 0)
-      (effects (font (size 1.27 1.27)) (justify left))
-    )
-    (property "Footprint" "" (id 2) (at 54.3052 93.98 0)
+    (property "Value" "100nF/50V" (id 1) (at 55.88 92.71 0)
+      (effects (font (size 1.27 1.27)) (justify left))
+    )
+    (property "Footprint" "Capacitor_SMD:C_0603_1608Metric" (id 2) (at 54.3052 93.98 0)
       (effects (font (size 1.27 1.27)) hide)
     )
@@
       (effects (font (size 1.27 1.27)) (justify left))
     )
-    (property "Value" "10uF" (id 1) (at 77.47 33.02 0)
-      (effects (font (size 1.27 1.27)) (justify left))
-    )
-    (property "Footprint" "" (id 2) (at 75.8952 34.29 0)
+    (property "Value" "10uF/25V" (id 1) (at 77.47 33.02 0)
+      (effects (font (size 1.27 1.27)) (justify left))
+    )
+    (property "Footprint" "Capacitor_SMD:C_1206_3216Metric" (id 2) (at 75.8952 34.29 0)
       (effects (font (size 1.27 1.27)) hide)
     )
@@
       (effects (font (size 1.27 1.27)) (justify left))
     )
-    (property "Value" "100nF" (id 1) (at 87.63 33.02 0)
-      (effects (font (size 1.27 1.27)) (justify left))
-    )
-    (property "Footprint" "" (id 2) (at 86.0552 34.29 0)
+    (property "Value" "100nF/50V" (id 1) (at 87.63 33.02 0)
+      (effects (font (size 1.27 1.27)) (justify left))
+    )
+    (property "Footprint" "Capacitor_SMD:C_0603_1608Metric" (id 2) (at 86.0552 34.29 0)
       (effects (font (size 1.27 1.27)) hide)
     )
@@
     (property "Reference" "C8" (id 0) (at 87.63 114.3 90))
     (property "Value" "20pF" (id 1) (at 87.63 116.84 90))
-    (property "Footprint" "" (id 2) (at 91.44 119.6848 0)
+    (property "Footprint" "Capacitor_SMD:C_0603_1608Metric" (id 2) (at 91.44 119.6848 0)
       (effects (font (size 1.27 1.27)) hide)
     )
@@
     (property "Reference" "C9" (id 0) (at 87.63 124.46 90))
     (property "Value" "20pF" (id 1) (at 87.63 127 90))
-    (property "Footprint" "" (id 2) (at 91.44 129.8448 0)
+    (property "Footprint" "Capacitor_SMD:C_0603_1608Metric" (id 2) (at 91.44 129.8448 0)
       (effects (font (size 1.27 1.27)) hide)
     )
@@
       (effects (font (size 1.27 1.27)) (justify left))
     )
-    (property "Value" "10uF" (id 1) (at 99.06 33.02 0)
-      (effects (font (size 1.27 1.27)) (justify left))
-    )
-    (property "Footprint" "" (id 2) (at 97.4852 34.29 0)
+    (property "Value" "10uF/25V" (id 1) (at 99.06 33.02 0)
+      (effects (font (size 1.27 1.27)) (justify left))
+    )
+    (property "Footprint" "Capacitor_SMD:C_1206_3216Metric" (id 2) (at 97.4852 34.29 0)
       (effects (font (size 1.27 1.27)) hide)
     )
@@
       (effects (font (size 1.27 1.27)) (justify left))
     )
-    (property "Value" "10uF" (id 1) (at 107.95 53.34 0)
-      (effects (font (size 1.27 1.27)) (justify left))
-    )
-    (property "Footprint" "" (id 2) (at 106.3752 54.61 0)
+    (property "Value" "10uF/25V" (id 1) (at 107.95 53.34 0)
+      (effects (font (size 1.27 1.27)) (justify left))
+    )
+    (property "Footprint" "Capacitor_SMD:C_1206_3216Metric" (id 2) (at 106.3752 54.61 0)
       (effects (font (size 1.27 1.27)) hide)
     )
@@
       (effects (font (size 1.27 1.27)) (justify left))
     )
-    (property "Value" "100nF" (id 1) (at 109.22 33.02 0)
-      (effects (font (size 1.27 1.27)) (justify left))
-    )
-    (property "Footprint" "" (id 2) (at 107.6452 34.29 0)
+    (property "Value" "100nF/50V" (id 1) (at 109.22 33.02 0)
+      (effects (font (size 1.27 1.27)) (justify left))
+    )
+    (property "Footprint" "Capacitor_SMD:C_0603_1608Metric" (id 2) (at 107.6452 34.29 0)
       (effects (font (size 1.27 1.27)) hide)
     )
@@
       (effects (font (size 1.27 1.27)) (justify left))
     )
-    (property "Value" "100nF" (id 1) (at 165.1 26.67 0)
-      (effects (font (size 1.27 1.27)) (justify left))
-    )
-    (property "Footprint" "" (id 2) (at 163.5252 27.94 0)
+    (property "Value" "100nF/50V" (id 1) (at 165.1 26.67 0)
+      (effects (font (size 1.27 1.27)) (justify left))
+    )
+    (property "Footprint" "Capacitor_SMD:C_0603_1608Metric" (id 2) (at 163.5252 27.94 0)
       (effects (font (size 1.27 1.27)) hide)
     )
@@
       (effects (font (size 1.27 1.27)) (justify left))
     )
-    (property "Value" "100nF" (id 1) (at 176.53 26.67 0)
-      (effects (font (size 1.27 1.27)) (justify left))
-    )
-    (property "Footprint" "" (id 2) (at 174.9552 27.94 0)
+    (property "Value" "100nF/50V" (id 1) (at 176.53 26.67 0)
+      (effects (font (size 1.27 1.27)) (justify left))
+    )
+    (property "Footprint" "Capacitor_SMD:C_0603_1608Metric" (id 2) (at 174.9552 27.94 0)
       (effects (font (size 1.27 1.27)) hide)
     )
@@
       (effects (font (size 1.27 1.27)) (justify left))
     )
-    (property "Value" "100nF" (id 1) (at 187.96 26.67 0)
-      (effects (font (size 1.27 1.27)) (justify left))
-    )
-    (property "Footprint" "" (id 2) (at 186.3852 27.94 0)
+    (property "Value" "100nF/50V" (id 1) (at 187.96 26.67 0)
+      (effects (font (size 1.27 1.27)) (justify left))
+    )
+    (property "Footprint" "Capacitor_SMD:C_0603_1608Metric" (id 2) (at 186.3852 27.94 0)
       (effects (font (size 1.27 1.27)) hide)
     )
@@
       (effects (font (size 1.27 1.27)) (justify left))
     )
-    (property "Value" "100nF" (id 1) (at 199.39 26.67 0)
-      (effects (font (size 1.27 1.27)) (justify left))
-    )
-    (property "Footprint" "" (id 2) (at 197.8152 27.94 0)
+    (property "Value" "100nF/50V" (id 1) (at 199.39 26.67 0)
+      (effects (font (size 1.27 1.27)) (justify left))
+    )
+    (property "Footprint" "Capacitor_SMD:C_0603_1608Metric" (id 2) (at 197.8152 27.94 0)
       (effects (font (size 1.27 1.27)) hide)
     )
@@
       (effects (font (size 1.27 1.27)) (justify left))
     )
-    (property "Value" "100nF" (id 1) (at 210.82 26.67 0)
-      (effects (font (size 1.27 1.27)) (justify left))
-    )
-    (property "Footprint" "" (id 2) (at 209.2452 27.94 0)
+    (property "Value" "100nF/50V" (id 1) (at 210.82 26.67 0)
+      (effects (font (size 1.27 1.27)) (justify left))
+    )
+    (property "Footprint" "Capacitor_SMD:C_0603_1608Metric" (id 2) (at 209.2452 27.94 0)
       (effects (font (size 1.27 1.27)) hide)
     )
@@
       (effects (font (size 1.27 1.27)) (justify left))
     )
-    (property "Value" "100nF" (id 1) (at 222.25 26.67 0)
-      (effects (font (size 1.27 1.27)) (justify left))
-    )
-    (property "Footprint" "" (id 2) (at 220.6752 27.94 0)
+    (property "Value" "100nF/50V" (id 1) (at 222.25 26.67 0)
+      (effects (font (size 1.27 1.27)) (justify left))
+    )
+    (property "Footprint" "Capacitor_SMD:C_0603_1608Metric" (id 2) (at 220.6752 27.94 0)
       (effects (font (size 1.27 1.27)) hide)
     )
@@
       (effects (font (size 1.27 1.27)) (justify left))
     )
-    (property "Value" "100nF" (id 1) (at 233.68 26.67 0)
-      (effects (font (size 1.27 1.27)) (justify left))
-    )
-    (property "Footprint" "" (id 2) (at 232.1052 27.94 0)
-      (effects (font (size 1.27 1.27)) hide)
-    )
+    (property "Value" "100nF/50V" (id 1) (at 233.68 26.67 0)
+      (effects (font (size 1.27 1.27)) (justify left))
+    )
+    (property "Footprint" "Capacitor_SMD:C_0603_1608Metric" (id 2) (at 232.1052 27.94 0)
+      (effects (font (size 1.27 1.27)) hide)
+    )

Commit message: placing test
Parts:
- L1, L2: footprint (none) -> Inductor_SMD:L_0603_1608Metric
- R13, R14, R15, R16, R17, R18, R19, R20: footprint (none) -> Resistor_SMD:R_0603_1608Metric
- U4: footprint (none) -> Package_SO:SO-8_3.9x4.9mm_P1.27mm
- Y1: footprint (none) -> Crystal:Crystal_SMD_0603-2Pin_6.0x3.5mm
Other:
- moved on the sheet: C10, C14, C15, C16, C17, C18, C19, C6, C7, L1, L2

Commit message: routing completed
Parts:
- removed Y1: 12MHz, Crystal:Crystal_SMD_0603-2Pin_6.0x3.5mm, symbol Device:Crystal
- added Y1: 12MHz, Crystal:Crystal_SMD_3225-4Pin_3.2x2.5mm, symbol Device:Crystal_GND24
Connections:
- net GND: now also Y1.2, Y1.4
- net ~RXLED: no longer R20.1, U2.55 (BCBUS4)
- net at C8.2, U2.2 (OSCI): now also Y1.3
- net at C9.2, U2.3 (OSCO): now also Y1.1
- new net ~TXLED: R20.1, U2.55 (BCBUS4)
Changed lines of the file:
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@@
   (junction (at 72.39 102.87) (diameter 0.9144) (color 0 0 0 0))
   (junction (at 74.93 19.05) (diameter 0.9144) (color 0 0 0 0))
+  (junction (at 83.82 125.73) (diameter 0.9144) (color 0 0 0 0))
   (junction (at 83.82 130.81) (diameter 0.9144) (color 0 0 0 0))
   (junction (at 91.44 24.13) (diameter 0.9144) (color 0 0 0 0))
@@
   (junction (at 152.4 31.75) (diameter 0.9144) (color 0 0 0 0))
   (junction (at 176.53 20.32) (diameter 0.9144) (color 0 0 0 0))
+  (no_connect (at 172.72 57.15))
+  (no_connect (at 172.72 74.93))
+  (no_connect (at 172.72 113.03))
+  (no_connect (at 172.72 128.27))
+  (no_connect (at 172.72 110.49))
+  (no_connect (at 172.72 135.89))
+  (no_connect (at 172.72 133.35))
+  (no_connect (at 172.72 52.07))
+  (no_connect (at 172.72 80.01))
+  (no_connect (at 172.72 59.69))
+  (no_connect (at 172.72 69.85))
+  (no_connect (at 172.72 125.73))
+  (no_connect (at 172.72 115.57))
+  (no_connect (at 172.72 64.77))
   (no_connect (at 172.72 67.31))
-  (no_connect (at 172.72 133.35))
-  (no_connect (at 172.72 125.73))
-  (no_connect (at 172.72 110.49))
-  (no_connect (at 172.72 74.93))
-  (no_connect (at 172.72 128.27))
-  (no_connect (at 172.72 135.89))
   (no_connect (at 172.72 77.47))
+  (no_connect (at 172.72 72.39))
   (no_connect (at 172.72 123.19))
   (no_connect (at 172.72 82.55))
-  (no_connect (at 172.72 72.39))
-  (no_connect (at 172.72 80.01))
-  (no_connect (at 172.72 113.03))
-  (no_connect (at 172.72 69.85))
-  (no_connect (at 172.72 59.69))
-  (no_connect (at 172.72 64.77))
-  (no_connect (at 172.72 57.15))
-  (no_connect (at 172.72 52.07))
-  (no_connect (at 172.72 115.57))
   (wire (pts (xy 19.05 100.33) (xy 27.94 100.33))
     (stroke (width 0) (type solid) (color 0 0 0 0))
@@
     (stroke (width 0) (type solid) (color 0 0 0 0))
   )
-  (wire (pts (xy 83.82 120.65) (xy 83.82 130.81))
+  (wire (pts (xy 83.82 120.65) (xy 83.82 125.73))
+    (stroke (width 0) (type solid) (color 0 0 0 0))
+  )
+  (wire (pts (xy 83.82 125.73) (xy 83.82 130.81))
+    (stroke (width 0) (type solid) (color 0 0 0 0))
+  )
+  (wire (pts (xy 83.82 125.73) (xy 91.44 125.73))
     (stroke (width 0) (type solid) (color 0 0 0 0))
   )
@@
   )
   (wire (pts (xy 101.6 113.03) (xy 111.76 113.03))
+    (stroke (width 0) (type solid) (color 0 0 0 0))
+  )
+  (wire (pts (xy 101.6 125.73) (xy 101.6 133.35))
     (stroke (width 0) (type solid) (color 0 0 0 0))
   )
@@
     (effects (font (size 1.27 1.27)) (justify right bottom))
   )
-  (label "~RXLED" (at 185.42 120.65 180)
+  (label "~TXLED" (at 185.42 120.65 180)
     (effects (font (size 1.27 1.27)) (justify right bottom))
   )
@@
     )
     (property "Datasheet" "" (id 3) (at 91.44 34.29 0)
+      (effects (font (size 1.27 1.27)) hide)
+    )
+  )
+  (symbol (lib_id "power:GND") (at 101.6 133.35 0) (unit 1)
+    (in_bom yes) (on_board yes)
+    (property "Reference" "#PWR0101" (id 0) (at 101.6 139.7 0)
+      (effects (font (size 1.27 1.27)) hide)
+    )
+    (property "Value" "GND" (id 1) (at 104.14 135.89 0))
+    (property "Footprint" "" (id 2) (at 101.6 133.35 0)
+      (effects (font (size 1.27 1.27)) hide)
+    )
+    (property "Datasheet" "" (id 3) (at 101.6 133.35 0)
       (effects (font (size 1.27 1.27)) hide)
     )
@@
     )
   )
-  (symbol (lib_id "Device:Crystal") (at 96.52 125.73 90) (unit 1)
-    (in_bom yes) (on_board yes)
-    (property "Reference" "Y1" (id 0) (at 100.33 124.46 90)
+  (symbol (lib_id "Device:Crystal_GND24") (at 96.52 125.73 90) (unit 1)
+    (in_bom yes) (on_board yes)
+    (property "Reference" "Y1" (id 0) (at 102.87 124.46 90)
       (effects (font (size 1.27 1.27)) (justify right))
     )
-    (property "Value" "12MHz" (id 1) (at 100.33 127 90)
+    (property "Value" "12MHz" (id 1) (at 102.87 127 90)
       (effects (font (size 1.27 1.27)) (justify right))
     )
-    (property "Footprint" "Crystal:Crystal_SMD_0603-2Pin_6.0x3.5mm" (id 2) (at 96.52 125.73 0)
-      (effects (font (size 1.27 1.27)) hide)
-    )
-    (property "Datasheet" "~" (id 3) (at 96.52 125.73 0)
-      (effects (font (size 1.27 1.27)) hide)
-    )
+    (property "Footprint" "Crystal:Crystal_SMD_3225-4Pin_3.2x2.5mm" (id 2) (at 96.52 125.73 0)
+      (effects (font (size 1.27 1.27)) hide)
+    )
+    (property "Datasheet" "https://ar.mouser.com/datasheet/2/96/008-0288-0_F-786189.pdf" (id 3) (at 96.52 125.73 0)
+      (effects (font (size 1.27 1.27)) hide)
+    )

Commit message: v0.1.0
Parts:
- C10, C11, C6: PN (none) -> CL31A106KAHNNNE
- C12, C13, C14, C15, C16, C17, C18, C19, C5, C7: PN (none) -> CL10B104KB8NNWC
- C8, C9: PN (none) -> 06035A200JAT2A
Changed lines of the file:
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@@
   (junction (at 152.4 31.75) (diameter 0.9144) (color 0 0 0 0))
   (junction (at 176.53 20.32) (diameter 0.9144) (color 0 0 0 0))
+  (no_connect (at 172.72 52.07))
   (no_connect (at 172.72 57.15))
-  (no_connect (at 172.72 74.93))
-  (no_connect (at 172.72 113.03))
-  (no_connect (at 172.72 128.27))
-  (no_connect (at 172.72 110.49))
-  (no_connect (at 172.72 135.89))
-  (no_connect (at 172.72 133.35))
-  (no_connect (at 172.72 52.07))
-  (no_connect (at 172.72 80.01))
   (no_connect (at 172.72 59.69))
-  (no_connect (at 172.72 69.85))
-  (no_connect (at 172.72 125.73))
-  (no_connect (at 172.72 115.57))
   (no_connect (at 172.72 64.77))
   (no_connect (at 172.72 67.31))
+  (no_connect (at 172.72 69.85))
+  (no_connect (at 172.72 72.39))
+  (no_connect (at 172.72 74.93))
   (no_connect (at 172.72 77.47))
-  (no_connect (at 172.72 72.39))
+  (no_connect (at 172.72 80.01))
+  (no_connect (at 172.72 82.55))
+  (no_connect (at 172.72 110.49))
+  (no_connect (at 172.72 113.03))
+  (no_connect (at 172.72 115.57))
   (no_connect (at 172.72 123.19))
-  (no_connect (at 172.72 82.55))
+  (no_connect (at 172.72 125.73))
+  (no_connect (at 172.72 128.27))
+  (no_connect (at 172.72 133.35))
+  (no_connect (at 172.72 135.89))
   (wire (pts (xy 19.05 100.33) (xy 27.94 100.33))
     (stroke (width 0) (type solid) (color 0 0 0 0))
@@
       (effects (font (size 1.27 1.27)) hide)
     )
+    (property "PN" "CL10B104KB8NNWC" (id 4) (at 53.34 90.17 0)
+      (effects (font (size 1.27 1.27)) hide)
+    )
   )
   (symbol (lib_id "Device:C") (at 59.69 30.48 0) (unit 1)
@@
       (effects (font (size 1.27 1.27)) hide)
     )
+    (property "PN" "CL31A106KAHNNNE" (id 4) (at 59.69 30.48 0)
+      (effects (font (size 1.27 1.27)) hide)
+    )
   )
   (symbol (lib_id "Device:C") (at 74.93 30.48 0) (unit 1)
@@
     )
     (property "Datasheet" "~" (id 3) (at 74.93 30.48 0)
+      (effects (font (size 1.27 1.27)) hide)
+    )
+    (property "PN" "CL10B104KB8NNWC" (id 4) (at 74.93 30.48 0)
       (effects (font (size 1.27 1.27)) hide)
     )
@@
       (effects (font (size 1.27 1.27)) hide)
     )
+    (property "PN" "06035A200JAT2A" (id 4) (at 87.63 120.65 0)
+      (effects (font (size 1.27 1.27)) hide)
+    )
   )
   (symbol (lib_id "Device:C") (at 87.63 130.81 90) (unit 1)
@@
       (effects (font (size 1.27 1.27)) hide)
     )
+    (property "PN" "06035A200JAT2A" (id 4) (at 87.63 130.81 0)
+      (effects (font (size 1.27 1.27)) hide)
+    )
   )
   (symbol (lib_id "Device:C") (at 91.44 30.48 0) (unit 1)
@@
       (effects (font (size 1.27 1.27)) hide)
     )
+    (property "PN" "CL31A106KAHNNNE" (id 4) (at 91.44 30.48 0)
+      (effects (font (size 1.27 1.27)) hide)
+    )
   )
   (symbol (lib_id "Device:C") (at 105.41 50.8 0) (unit 1)
@@
       (effects (font (size 1.27 1.27)) hide)
     )
+    (property "PN" "CL31A106KAHNNNE" (id 4) (at 105.41 50.8 0)
+      (effects (font (size 1.27 1.27)) hide)
+    )
   )
   (symbol (lib_id "Device:C") (at 106.68 30.48 0) (unit 1)
@@
       (effects (font (size 1.27 1.27)) hide)
     )
+    (property "PN" "CL10B104KB8NNWC" (id 4) (at 106.68 30.48 0)
+      (effects (font (size 1.27 1.27)) hide)
+    )
   )
   (symbol (lib_id "Device:C") (at 162.56 24.13 0) (unit 1)
@@
       (effects (font (size 1.27 1.27)) hide)
     )
+    (property "PN" "CL10B104KB8NNWC" (id 4) (at 162.56 24.13 0)
+      (effects (font (size 1.27 1.27)) hide)
+    )
   )
   (symbol (lib_id "Device:C") (at 176.53 24.13 0) (unit 1)
@@
       (effects (font (size 1.27 1.27)) hide)
     )
+    (property "PN" "CL10B104KB8NNWC" (id 4) (at 176.53 24.13 0)
+      (effects (font (size 1.27 1.27)) hide)
+    )
   )
   (symbol (lib_id "Device:C") (at 190.5 24.13 0) (unit 1)
@@
       (effects (font (size 1.27 1.27)) hide)
     )
+    (property "PN" "CL10B104KB8NNWC" (id 4) (at 190.5 24.13 0)
+      (effects (font (size 1.27 1.27)) hide)
+    )
   )
   (symbol (lib_id "Device:C") (at 208.28 24.13 0) (unit 1)
@@
       (effects (font (size 1.27 1.27)) hide)
     )
+    (property "PN" "CL10B104KB8NNWC" (id 4) (at 208.28 24.13 0)
+      (effects (font (size 1.27 1.27)) hide)
+    )
   )
   (symbol (lib_id "Device:C") (at 223.52 24.13 0) (unit 1)
@@
       (effects (font (size 1.27 1.27)) hide)
     )
+    (property "PN" "CL10B104KB8NNWC" (id 4) (at 223.52 24.13 0)
+      (effects (font (size 1.27 1.27)) hide)
+    )
   )
   (symbol (lib_id "Device:C") (at 238.76 24.13 0) (unit 1)
@@
       (effects (font (size 1.27 1.27)) hide)
     )
+    (property "PN" "CL10B104KB8NNWC" (id 4) (at 238.76 24.13 0)
+      (effects (font (size 1.27 1.27)) hide)
+    )
   )
   (symbol (lib_id "Device:C") (at 254 24.13 0) (unit 1)
@@
       (effects (font (size 1.27 1.27)) hide)
     )
+    (property "PN" "CL10B104KB8NNWC" (id 4) (at 254 24.13 0)
+      (effects (font (size 1.27 1.27)) hide)
+    )
