File: ft2232.kicad_sch (KiCad schematic)
At the start: 30 parts, among them U2 FT2232HL, U4 93C46, Y1 12MHz

Commit message: add PN
Parts:
- D3, D4: PN (none) -> 598-8070-107F
- L1, L2: value HZ0805E601R-10 -> MPZ1608S102ATA00; PN (none) -> MPZ1608S102ATA00
- R13, R14, R16: PN (none) -> CRCW060310K0FKEBC
- R15, R19, R20: PN (none) -> CRCW06032K20FKEB
- R17: PN (none) -> RMCF0603FT12K0
- R18: PN (none) -> RMCF0603FT1K00
- U2: PN (none) -> FT2232HL-REEL
- U4: value 93C46 -> 93LC46B; PN (none) -> 93LC46B
- Y1: PN (none) -> 403C11A12M00000
Changed lines of the file:
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@@
+      (effects (font (size 1.27 1.27)) hide)
+    )
+    (property "PN" "CRCW060310K0FKEBC" (id 4) (at 27.94 95.25 0)
       (effects (font (size 1.27 1.27)) hide)
     )
@@
     )
     (property "Datasheet" "~" (id 3) (at 64.77 95.25 0)
+      (effects (font (size 1.27 1.27)) hide)
+    )
+    (property "PN" "CRCW060310K0FKEBC" (id 4) (at 64.77 95.25 0)
       (effects (font (size 1.27 1.27)) hide)
     )
@@
       (effects (font (size 1.27 1.27)) hide)
     )
+    (property "PN" "CRCW06032K20FKEB" (id 4) (at 68.58 102.87 0)
+      (effects (font (size 1.27 1.27)) hide)
+    )
   )
   (symbol (lib_id "Device:R") (at 72.39 95.25 0) (unit 1)
@@
     )
     (property "Datasheet" "~" (id 3) (at 72.39 95.25 0)
+      (effects (font (size 1.27 1.27)) hide)
+    )
+    (property "PN" "CRCW060310K0FKEBC" (id 4) (at 72.39 95.25 0)
       (effects (font (size 1.27 1.27)) hide)
     )
@@
       (effects (font (size 1.27 1.27)) hide)
     )
+    (property "PN" "RMCF0603FT12K0" (id 4) (at 101.6 74.93 0)
+      (effects (font (size 1.27 1.27)) hide)
+    )
   )
   (symbol (lib_id "Device:R") (at 107.95 80.01 90) (unit 1)
@@
       (effects (font (size 1.27 1.27)) hide)
     )
+    (property "PN" "RMCF0603FT1K00" (id 4) (at 107.95 80.01 0)
+      (effects (font (size 1.27 1.27)) hide)
+    )
   )
   (symbol (lib_id "Device:R") (at 194.31 118.11 90) (unit 1)
@@
       (effects (font (size 1.27 1.27)) hide)
     )
+    (property "PN" "CRCW06032K20FKEB" (id 4) (at 194.31 118.11 0)
+      (effects (font (size 1.27 1.27)) hide)
+    )
   )
   (symbol (lib_id "Device:R") (at 194.31 127 90) (unit 1)
@@
       (effects (font (size 1.27 1.27)) hide)
     )
+    (property "PN" "CRCW06032K20FKEB" (id 4) (at 194.31 127 0)
+      (effects (font (size 1.27 1.27)) hide)
+    )
   )
   (symbol (lib_id "pspice:INDUCTOR") (at 45.72 19.05 0) (unit 1)
     (in_bom yes) (on_board yes)
     (property "Reference" "L1" (id 0) (at 38.1 17.78 0))
-    (property "Value" "HZ0805E601R-10" (id 1) (at 45.72 20.32 0))
+    (property "Value" "MPZ1608S102ATA00" (id 1) (at 45.72 20.32 0))
     (property "Footprint" "Inductor_SMD:L_0603_1608Metric" (id 2) (at 45.72 19.05 0)
       (effects (font (size 1.27 1.27)) hide)
@@
       (effects (font (size 1.27 1.27)) hide)
     )
+    (property "PN" "MPZ1608S102ATA00" (id 4) (at 45.72 19.05 0)
+      (effects (font (size 1.27 1.27)) hide)
+    )
   )
   (symbol (lib_id "pspice:INDUCTOR") (at 45.72 24.13 0) (unit 1)
     (in_bom yes) (on_board yes)
     (property "Reference" "L2" (id 0) (at 38.1 22.86 0))
-    (property "Value" "HZ0805E601R-10" (id 1) (at 45.72 25.4 0))
+    (property "Value" "MPZ1608S102ATA00" (id 1) (at 45.72 25.4 0))
     (property "Footprint" "Inductor_SMD:L_0603_1608Metric" (id 2) (at 45.72 24.13 0)
       (effects (font (size 1.27 1.27)) hide)
     )
     (property "Datasheet" "~" (id 3) (at 45.72 24.13 0)
+      (effects (font (size 1.27 1.27)) hide)
+    )
+    (property "PN" "MPZ1608S102ATA00" (id 4) (at 45.72 24.13 0)
       (effects (font (size 1.27 1.27)) hide)
     )
@@
       (effects (font (size 1.27 1.27)) hide)
     )
+    (property "PN" "598-8070-107F" (id 4) (at 201.93 118.11 0)
+      (effects (font (size 1.27 1.27)) hide)
+    )
   )
   (symbol (lib_id "Device:LED") (at 201.93 127 0) (unit 1)
@@
       (effects (font (size 1.27 1.27)) hide)
     )
+    (property "PN" "598-8070-107F" (id 4) (at 201.93 127 0)
+      (effects (font (size 1.27 1.27)) hide)
+    )
   )
   (symbol (lib_id "Device:C") (at 53.34 90.17 0) (unit 1)
@@
       (effects (font (size 1.27 1.27)) hide)
     )
+    (property "PN" "403C11A12M00000" (id 4) (at 96.52 125.73 0)
+      (effects (font (size 1.27 1.27)) hide)
+    )
   )
   (symbol (lib_id "Memory_EEPROM:93CxxC") (at 41.91 102.87 0) (unit 1)
     (in_bom yes) (on_board yes)
     (property "Reference" "U4" (id 0) (at 46.99 93.98 0))
-    (property "Value" "93C46" (id 1) (at 46.99 96.52 0))
+    (property "Value" "93LC46B" (id 1) (at 46.99 96.52 0))
     (property "Footprint" "Package_SO:SO-8_3.9x4.9mm_P1.27mm" (id 2) (at 41.91 102.87 0)
       (effects (font (size 1.27 1.27)) hide)
     )
     (property "Datasheet" "http://ww1.microchip.com/downloads/en/DeviceDoc/20001749K.pdf" (id 3) (at 41.91 102.87 0)
+      (effects (font (size 1.27 1.27)) hide)
+    )
+    (property "PN" "93LC46B" (id 4) (at 41.91 102.87 0)
       (effects (font (size 1.27 1.27)) hide)
     )
@@
       (effects (font (size 1.27 1.27)) hide)
     )
+    (property "PN" "FT2232HL-REEL" (id 4) (at 142.24 90.17 0)
+      (effects (font (size 1.27 1.27)) hide)
+    )
