File: esp-wroom-32.kicad_sch (KiCad schematic)
At the start: 1 part, among them U1 ESP32-WROOM-32

Commit message: erc ok
Parts:
- added C20, C22: 100nF, symbol Device:C
- added C21: 22uF, symbol Device:C
- added R21: 10k, symbol Device:R
Connections:
- net GND: now reaches U1.1 (GND), U1.15 (GND), U1.38 (GND), U1.39 (GND)
- net GND: now also C20.2, C21.2, C22.2
- net IO25: now reaches U1.10 (IO25)
- net IO26: now reaches U1.11 (IO26)
- net IO27: now reaches U1.12 (IO27)
- net IO14: now reaches U1.13 (IO14)
- net IO12: now reaches U1.14 (IO12)
- net IO13: now reaches U1.16 (IO13)
- net SD2: now reaches U1.17 (SHD/SD2)
- net SD3: now reaches U1.18 (SWP/SD3)
- net CMD: now reaches U1.19 (SCS/CMD)
- net +3V3: now reaches U1.2 (VDD)
- net +3V3: now also C21.1, C22.1, R21.1
- net CLK: now reaches U1.20 (SCK/CLK)
- net SD0: now reaches U1.21 (SDO/SD0)
- net SD1: now reaches U1.22 (SDI/SD1)
- net IO15: now reaches U1.23 (IO15)
- net IO2: now reaches U1.24 (IO2)
- net IO0: now reaches U1.25 (IO0)
- net IO4: now reaches U1.26 (IO4)
- net IO16: now reaches U1.27 (IO16)
- net IO17: now reaches U1.28 (IO17)
- net IO5: now reaches U1.29 (IO5)
- net EN: now reaches U1.3 (EN)
- net EN: now also C20.1, R21.2
- net IO18: now reaches U1.30 (IO18)
- net IO19: now reaches U1.31 (IO19)
- net IO21: now reaches U1.33 (IO21)
- net RXD0: now reaches U1.34 (RXD0/IO3)
- net TXD0: now reaches U1.35 (TXD0/IO1)
- net IO22: now reaches U1.36 (IO22)
- net IO23: now reaches U1.37 (IO23)
- net SENSOR_VP: now reaches U1.4 (SENSOR_VP)
- net SENSOR_VN: now reaches U1.5 (SENSOR_VN)
- net IO34: now reaches U1.6 (IO34)
- net IO35: now reaches U1.7 (IO35)
- net IO32: now reaches U1.8 (IO32)
- net IO33: now reaches U1.9 (IO33)

Commit message: wip footprint assoc
Parts:
- C20, C22: value 100nF -> 100nF/50V; footprint (none) -> Capacitor_SMD:C_0603_1608Metric
- C21: value 22uF -> 10uF/25V; footprint (none) -> Capacitor_SMD:C_1206_3216Metric
Other:
- moved on the sheet: C21
Changed lines of the file:
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@@
     )
   )
-  (symbol (lib_id "power:+3V3") (at 111.76 34.29 0) (unit 1)
+  (symbol (lib_id "power:+3V3") (at 105.41 34.29 0) (unit 1)
     (in_bom yes) (on_board yes)
-    (property "Reference" "#PWR052" (id 0) (at 111.76 38.1 0)
+    (property "Reference" "#PWR052" (id 0) (at 105.41 38.1 0)
       (effects (font (size 1.27 1.27)) hide)
     )
-    (property "Value" "+3V3" (id 1) (at 113.03 29.21 0))
-    (property "Footprint" "" (id 2) (at 111.76 34.29 0)
+    (property "Value" "+3V3" (id 1) (at 106.68 29.21 0))
+    (property "Footprint" "" (id 2) (at 105.41 34.29 0)
       (effects (font (size 1.27 1.27)) hide)
     )
-    (property "Datasheet" "" (id 3) (at 111.76 34.29 0)
+    (property "Datasheet" "" (id 3) (at 105.41 34.29 0)
       (effects (font (size 1.27 1.27)) hide)
     )
@@
     )
   )
-  (symbol (lib_id "power:GND") (at 111.76 41.91 0) (unit 1)
+  (symbol (lib_id "power:GND") (at 105.41 41.91 0) (unit 1)
     (in_bom yes) (on_board yes)
-    (property "Reference" "#PWR053" (id 0) (at 111.76 48.26 0)
+    (property "Reference" "#PWR053" (id 0) (at 105.41 48.26 0)
       (effects (font (size 1.27 1.27)) hide)
     )
-    (property "Value" "GND" (id 1) (at 114.3 44.45 0))
-    (property "Footprint" "" (id 2) (at 111.76 41.91 0)
+    (property "Value" "GND" (id 1) (at 107.95 44.45 0))
+    (property "Footprint" "" (id 2) (at 105.41 41.91 0)
       (effects (font (size 1.27 1.27)) hide)
     )
-    (property "Datasheet" "" (id 3) (at 111.76 41.91 0)
+    (property "Datasheet" "" (id 3) (at 105.41 41.91 0)
       (effects (font (size 1.27 1.27)) hide)
     )
@@
       (effects (font (size 1.27 1.27)) (justify left))
     )
-    (property "Value" "100nF" (id 1) (at 76.2 53.34 0)
+    (property "Value" "100nF/50V" (id 1) (at 76.2 53.34 0)
       (effects (font (size 1.27 1.27)) (justify left))
     )
-    (property "Footprint" "" (id 2) (at 73.3552 55.88 0)
+    (property "Footprint" "Capacitor_SMD:C_0603_1608Metric" (id 2) (at 73.3552 55.88 0)
       (effects (font (size 1.27 1.27)) hide)
     )
@@
     )
   )
-  (symbol (lib_id "Device:C") (at 111.76 38.1 0) (unit 1)
+  (symbol (lib_id "Device:C") (at 105.41 38.1 0) (unit 1)
     (in_bom yes) (on_board yes)
-    (property "Reference" "C21" (id 0) (at 115.57 36.83 0)
+    (property "Reference" "C21" (id 0) (at 109.22 36.83 0)
       (effects (font (size 1.27 1.27)) (justify left))
     )
-    (property "Value" "22uF" (id 1) (at 115.57 39.37 0)
+    (property "Value" "10uF/25V" (id 1) (at 109.22 39.37 0)
       (effects (font (size 1.27 1.27)) (justify left))
     )
-    (property "Footprint" "" (id 2) (at 112.7252 41.91 0)
+    (property "Footprint" "Capacitor_SMD:C_1206_3216Metric" (id 2) (at 106.3752 41.91 0)
       (effects (font (size 1.27 1.27)) hide)
     )
-    (property "Datasheet" "~" (id 3) (at 111.76 38.1 0)
+    (property "Datasheet" "~" (id 3) (at 105.41 38.1 0)
       (effects (font (size 1.27 1.27)) hide)
     )
@@
       (effects (font (size 1.27 1.27)) (justify left))
     )
-    (property "Value" "100nF" (id 1) (at 127 39.37 0)
+    (property "Value" "100nF/50V" (id 1) (at 127 39.37 0)
       (effects (font (size 1.27 1.27)) (justify left))
     )
-    (property "Footprint" "" (id 2) (at 124.1552 41.91 0)
+    (property "Footprint" "Capacitor_SMD:C_0603_1608Metric" (id 2) (at 124.1552 41.91 0)
       (effects (font (size 1.27 1.27)) hide)
     )

Commit message: placing test
Parts:
- R21: footprint (none) -> Resistor_SMD:R_0603_1608Metric
Changed lines of the file:
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@@
       (effects (font (size 1.27 1.27)) (justify left))
     )
-    (property "Footprint" "" (id 2) (at 70.612 41.91 90)
+    (property "Footprint" "Resistor_SMD:R_0603_1608Metric" (id 2) (at 70.612 41.91 90)
       (effects (font (size 1.27 1.27)) hide)
     )

Commit message: sch update
Other:
- moved on the sheet: C21, C22
Changed lines of the file:
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@@
     )
   )
-  (symbol (lib_id "power:+3V3") (at 105.41 34.29 0) (unit 1)
+  (symbol (lib_id "power:+3V3") (at 100.33 30.48 0) (unit 1)
     (in_bom yes) (on_board yes)
-    (property "Reference" "#PWR052" (id 0) (at 105.41 38.1 0)
+    (property "Reference" "#PWR052" (id 0) (at 100.33 34.29 0)
       (effects (font (size 1.27 1.27)) hide)
     )
-    (property "Value" "+3V3" (id 1) (at 106.68 29.21 0))
-    (property "Footprint" "" (id 2) (at 105.41 34.29 0)
+    (property "Value" "+3V3" (id 1) (at 101.6 25.4 0))
+    (property "Footprint" "" (id 2) (at 100.33 30.48 0)
       (effects (font (size 1.27 1.27)) hide)
     )
-    (property "Datasheet" "" (id 3) (at 105.41 34.29 0)
+    (property "Datasheet" "" (id 3) (at 100.33 30.48 0)
       (effects (font (size 1.27 1.27)) hide)
     )
   )
-  (symbol (lib_id "power:+3V3") (at 123.19 34.29 0) (unit 1)
+  (symbol (lib_id "power:+3V3") (at 118.11 30.48 0) (unit 1)
     (in_bom yes) (on_board yes)
-    (property "Reference" "#PWR054" (id 0) (at 123.19 38.1 0)
+    (property "Reference" "#PWR054" (id 0) (at 118.11 34.29 0)
       (effects (font (size 1.27 1.27)) hide)
     )
-    (property "Value" "+3V3" (id 1) (at 124.46 29.21 0))
-    (property "Footprint" "" (id 2) (at 123.19 34.29 0)
+    (property "Value" "+3V3" (id 1) (at 119.38 25.4 0))
+    (property "Footprint" "" (id 2) (at 118.11 30.48 0)
       (effects (font (size 1.27 1.27)) hide)
     )
-    (property "Datasheet" "" (id 3) (at 123.19 34.29 0)
+    (property "Datasheet" "" (id 3) (at 118.11 30.48 0)
       (effects (font (size 1.27 1.27)) hide)
     )
@@
     )
   )
-  (symbol (lib_id "power:GND") (at 105.41 41.91 0) (unit 1)
+  (symbol (lib_id "power:GND") (at 100.33 38.1 0) (unit 1)
     (in_bom yes) (on_board yes)
-    (property "Reference" "#PWR053" (id 0) (at 105.41 48.26 0)
+    (property "Reference" "#PWR053" (id 0) (at 100.33 44.45 0)
       (effects (font (size 1.27 1.27)) hide)
     )
-    (property "Value" "GND" (id 1) (at 107.95 44.45 0))
-    (property "Footprint" "" (id 2) (at 105.41 41.91 0)
+    (property "Value" "GND" (id 1) (at 102.87 40.64 0))
+    (property "Footprint" "" (id 2) (at 100.33 38.1 0)
       (effects (font (size 1.27 1.27)) hide)
     )
-    (property "Datasheet" "" (id 3) (at 105.41 41.91 0)
+    (property "Datasheet" "" (id 3) (at 100.33 38.1 0)
       (effects (font (size 1.27 1.27)) hide)
     )
   )
-  (symbol (lib_id "power:GND") (at 123.19 41.91 0) (unit 1)
+  (symbol (lib_id "power:GND") (at 118.11 38.1 0) (unit 1)
     (in_bom yes) (on_board yes)
-    (property "Reference" "#PWR055" (id 0) (at 123.19 48.26 0)
+    (property "Reference" "#PWR055" (id 0) (at 118.11 44.45 0)
       (effects (font (size 1.27 1.27)) hide)
     )
-    (property "Value" "GND" (id 1) (at 125.73 44.45 0))
-    (property "Footprint" "" (id 2) (at 123.19 41.91 0)
+    (property "Value" "GND" (id 1) (at 120.65 40.64 0))
+    (property "Footprint" "" (id 2) (at 118.11 38.1 0)
       (effects (font (size 1.27 1.27)) hide)
     )
-    (property "Datasheet" "" (id 3) (at 123.19 41.91 0)
+    (property "Datasheet" "" (id 3) (at 118.11 38.1 0)
       (effects (font (size 1.27 1.27)) hide)
     )
@@
     )
   )
-  (symbol (lib_id "Device:C") (at 105.41 38.1 0) (unit 1)
+  (symbol (lib_id "Device:C") (at 100.33 34.29 0) (unit 1)
     (in_bom yes) (on_board yes)
-    (property "Reference" "C21" (id 0) (at 109.22 36.83 0)
+    (property "Reference" "C21" (id 0) (at 104.14 33.02 0)
       (effects (font (size 1.27 1.27)) (justify left))
     )
-    (property "Value" "10uF/25V" (id 1) (at 109.22 39.37 0)
+    (property "Value" "10uF/25V" (id 1) (at 104.14 35.56 0)
       (effects (font (size 1.27 1.27)) (justify left))
     )
-    (property "Footprint" "Capacitor_SMD:C_1206_3216Metric" (id 2) (at 106.3752 41.91 0)
+    (property "Footprint" "Capacitor_SMD:C_1206_3216Metric" (id 2) (at 101.2952 38.1 0)
       (effects (font (size 1.27 1.27)) hide)
     )
-    (property "Datasheet" "~" (id 3) (at 105.41 38.1 0)
+    (property "Datasheet" "~" (id 3) (at 100.33 34.29 0)
       (effects (font (size 1.27 1.27)) hide)
     )
   )
-  (symbol (lib_id "Device:C") (at 123.19 38.1 0) (unit 1)
+  (symbol (lib_id "Device:C") (at 118.11 34.29 0) (unit 1)
     (in_bom yes) (on_board yes)
-    (property "Reference" "C22" (id 0) (at 127 36.83 0)
+    (property "Reference" "C22" (id 0) (at 121.92 33.02 0)
       (effects (font (size 1.27 1.27)) (justify left))
     )
-    (property "Value" "100nF/50V" (id 1) (at 127 39.37 0)
+    (property "Value" "100nF/50V" (id 1) (at 121.92 35.56 0)
       (effects (font (size 1.27 1.27)) (justify left))
     )
-    (property "Footprint" "Capacitor_SMD:C_0603_1608Metric" (id 2) (at 124.1552 41.91 0)
+    (property "Footprint" "Capacitor_SMD:C_0603_1608Metric" (id 2) (at 119.0752 38.1 0)
       (effects (font (size 1.27 1.27)) hide)
     )
-    (property "Datasheet" "~" (id 3) (at 123.19 38.1 0)
+    (property "Datasheet" "~" (id 3) (at 118.11 34.29 0)
       (effects (font (size 1.27 1.27)) hide)
     )

Commit message: v0.1.0
Parts:
- C20, C22: PN (none) -> CL10B104KB8NNWC
- C21: PN (none) -> CL31A106KAHNNNE
Changed lines of the file:
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@@
+      (effects (font (size 1.27 1.27)) hide)
+    )
+    (property "PN" "CL10B104KB8NNWC" (id 4) (at 72.39 52.07 0)
       (effects (font (size 1.27 1.27)) hide)
     )
@@
       (effects (font (size 1.27 1.27)) hide)
     )
+    (property "PN" "CL31A106KAHNNNE" (id 4) (at 100.33 34.29 0)
+      (effects (font (size 1.27 1.27)) hide)
+    )
   )
   (symbol (lib_id "Device:C") (at 118.11 34.29 0) (unit 1)
@@
       (effects (font (size 1.27 1.27)) hide)
     )
+    (property "PN" "CL10B104KB8NNWC" (id 4) (at 118.11 34.29 0)
+      (effects (font (size 1.27 1.27)) hide)
+    )

Commit message: add PN
Parts:
- R21: PN (none) -> CRCW060310K0FKEBC
- U1: PN (none) -> ESP32-WROOM-32E
Changed lines of the file:
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@@
+      (effects (font (size 1.27 1.27)) hide)
+    )
+    (property "PN" "CRCW060310K0FKEBC" (id 4) (at 72.39 41.91 0)
       (effects (font (size 1.27 1.27)) hide)
     )
@@
       (effects (font (size 1.27 1.27)) hide)
     )
+    (property "PN" "ESP32-WROOM-32E" (id 4) (at 135.89 81.28 0)
+      (effects (font (size 1.27 1.27)) hide)
+    )
