File: lisa32.kicad_sch (KiCad schematic)
At the start: 34 parts, among them J1 USB4105-GF-A, J2 Conn_01x19, J3 Conn_01x19, Q1 SS8050-G, Q2 SS8050-G, SW1 BOOT, SW2 RST, U3 LD1117S33TR_SOT223

Commit message: add PN
Parts:
- D5: PN (none) -> COM-11821
- J1: PN (none) -> USB4105-GF-A
- Q1, Q2: PN (none) -> SS8050-G
- R1: PN (none) -> CRGCQ0603J1M0
- R10, R11, R12, R23, R6, R7, R8, R9: PN (none) -> RMCF0603FT1K00
- R2, R3: PN (none) -> CRCW06035K10FKEBC
- R22: PN (none) -> RMCF0603FT150R
- R4, R5: PN (none) -> CRCW060310K0FKEBC
- SW1, SW2: PN (none) -> B3U-1000P
- U3: PN (none) -> LD1117S33TR
Changed lines of the file:
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@@
+      (effects (font (size 1.27 1.27)) hide)
+    )
+    (property "PN" "CRGCQ0603J1M0" (id 4) (at 29.21 81.28 0)
       (effects (font (size 1.27 1.27)) hide)
     )
@@
       (effects (font (size 1.27 1.27)) hide)
     )
+    (property "PN" "RMCF0603FT1K00" (id 4) (at 33.02 179.07 0)
+      (effects (font (size 1.27 1.27)) hide)
+    )
   )
   (symbol (lib_id "Device:R") (at 46.99 132.08 90) (unit 1)
@@
       (effects (font (size 1.27 1.27)) hide)
     )
+    (property "PN" "CRCW060310K0FKEBC" (id 4) (at 46.99 132.08 0)
+      (effects (font (size 1.27 1.27)) hide)
+    )
   )
   (symbol (lib_id "Device:R") (at 46.99 148.59 90) (unit 1)
@@
       (effects (font (size 1.27 1.27)) hide)
     )
+    (property "PN" "CRCW060310K0FKEBC" (id 4) (at 46.99 148.59 0)
+      (effects (font (size 1.27 1.27)) hide)
+    )
   )
   (symbol (lib_id "Device:R") (at 53.34 166.37 90) (unit 1)
@@
       (effects (font (size 1.27 1.27)) hide)
     )
+    (property "PN" "RMCF0603FT150R" (id 4) (at 53.34 166.37 0)
+      (effects (font (size 1.27 1.27)) hide)
+    )
   )
   (symbol (lib_id "Device:R") (at 60.96 41.91 90) (unit 1)
@@
       (effects (font (size 1.27 1.27)) hide)
     )
+    (property "PN" "CRCW06035K10FKEBC" (id 4) (at 60.96 41.91 0)
+      (effects (font (size 1.27 1.27)) hide)
+    )
   )
   (symbol (lib_id "Device:R") (at 60.96 44.45 90) (unit 1)
@@
       (effects (font (size 1.27 1.27)) hide)
     )
+    (property "PN" "CRCW06035K10FKEBC" (id 4) (at 60.96 44.45 0)
+      (effects (font (size 1.27 1.27)) hide)
+    )
   )
   (symbol (lib_id "Device:R") (at 180.34 25.4 90) (unit 1)
@@
       (effects (font (size 1.27 1.27)) hide)
     )
+    (property "PN" "RMCF0603FT1K00" (id 4) (at 180.34 25.4 0)
+      (effects (font (size 1.27 1.27)) hide)
+    )
   )
   (symbol (lib_id "Device:R") (at 180.34 27.94 90) (unit 1)
@@
       (effects (font (size 1.27 1.27)) hide)
     )
+    (property "PN" "RMCF0603FT1K00" (id 4) (at 180.34 27.94 0)
+      (effects (font (size 1.27 1.27)) hide)
+    )
   )
   (symbol (lib_id "Device:R") (at 180.34 50.8 90) (unit 1)
@@
       (effects (font (size 1.27 1.27)) hide)
     )
+    (property "PN" "RMCF0603FT1K00" (id 4) (at 180.34 50.8 0)
+      (effects (font (size 1.27 1.27)) hide)
+    )
   )
   (symbol (lib_id "Device:R") (at 180.34 53.34 90) (unit 1)
@@
       (effects (font (size 1.27 1.27)) hide)
     )
+    (property "PN" "RMCF0603FT1K00" (id 4) (at 180.34 53.34 0)
+      (effects (font (size 1.27 1.27)) hide)
+    )
   )
   (symbol (lib_id "Device:R") (at 180.34 55.88 90) (unit 1)
@@
       (effects (font (size 1.27 1.27)) hide)
     )
+    (property "PN" "RMCF0603FT1K00" (id 4) (at 180.34 55.88 0)
+      (effects (font (size 1.27 1.27)) hide)
+    )
   )
   (symbol (lib_id "Device:R") (at 180.34 58.42 90) (unit 1)
@@
       (effects (font (size 1.27 1.27)) hide)
     )
+    (property "PN" "RMCF0603FT1K00" (id 4) (at 180.34 58.42 0)
+      (effects (font (size 1.27 1.27)) hide)
+    )
   )
   (symbol (lib_id "Device:R") (at 180.34 60.96 90) (unit 1)
@@
       (effects (font (size 1.27 1.27)) hide)
     )
+    (property "PN" "RMCF0603FT1K00" (id 4) (at 180.34 60.96 0)
+      (effects (font (size 1.27 1.27)) hide)
+    )
   )
   (symbol (lib_id "Device:D_Schottky") (at 60.96 36.83 180) (unit 1)
@@
       (effects (font (size 1.27 1.27)) hide)
     )
+    (property "PN" "B3U-1000P" (id 4) (at 227.33 142.24 0)
+      (effects (font (size 1.27 1.27)) hide)
+    )
   )
   (symbol (lib_id "Switch:SW_Push") (at 256.54 142.24 0) (unit 1)
@@
       (effects (font (size 1.27 1.27)) hide)
     )
+    (property "PN" "B3U-1000P" (id 4) (at 256.54 142.24 0)
+      (effects (font (size 1.27 1.27)) hide)
+    )
   )
   (symbol (lib_id "Transistor_BJT:BC817") (at 59.69 132.08 0) (unit 1)
@@
       (effects (font (size 1.27 1.27)) (justify left) hide)
     )
+    (property "PN" "SS8050-G" (id 4) (at 59.69 132.08 0)
+      (effects (font (size 1.27 1.27)) hide)
+    )
   )
   (symbol (lib_id "Transistor_BJT:BC817") (at 59.69 148.59 0) (mirror x) (unit 1)
@@
     (property "Datasheet" "https://www.onsemi.com/pub/Collateral/BC818-D.pdf" (id 3) (at 59.69 148.59 0)
       (effects (font (size 1.27 1.27)) (justify left) hide)
+    )
+    (property "PN" "SS8050-G" (id 4) (at 59.69 148.59 0)
+      (effects (font (size 1.27 1.27)) hide)
     )
   )
@@
       (effects (font (size 1.27 1.27)) hide)
     )
+    (property "PN" "LD1117S33TR" (id 4) (at 49.53 102.87 0)
+      (effects (font (size 1.27 1.27)) hide)
+    )
   )
   (symbol (lib_id "LED:WS2812") (at 49.53 179.07 0) (unit 1)
@@
     (property "Datasheet" "https://cdn-shop.adafruit.com/datasheets/WS2812.pdf" (id 3) (at 52.07 188.595 0)
       (effects (font (size 1.27 1.27)) (justify left top) hide)
+    )
+    (property "PN" "COM-11821" (id 4) (at 49.53 179.07 0)
+      (effects (font (size 1.27 1.27)) hide)
     )
   )
@@
     )
     (property "Datasheet" "https://www.usb.org/sites/default/files/documents/usb_type-c.zip" (id 3) (at 40.64 52.07 0)
+      (effects (font (size 1.27 1.27)) hide)
+    )
+    (property "PN" "USB4105-GF-A" (id 4) (at 36.83 52.07 0)
       (effects (font (size 1.27 1.27)) hide)
     )
@@
     )
     (path "/5f304c88-142b-41d9-b86f-2d4158492d4d/8e4e4bab-8238-4376-9a74-f5c3e44fac11"
-      (reference "L1") (unit 1) (value "HZ0805E601R-10") (footprint "Inductor_SMD:L_0603_1608Metric")
+      (reference "L1") (unit 1) (value "MPZ1608S102ATA00") (footprint "Inductor_SMD:L_0603_1608Metric")
     )
     (path "/5f304c88-142b-41d9-b86f-2d4158492d4d/68c6a525-a215-4513-b1e7-64042ff0af7b"
-      (reference "L2") (unit 1) (value "HZ0805E601R-10") (footprint "Inductor_SMD:L_0603_1608Metric")
+      (reference "L2") (unit 1) (value "MPZ1608S102ATA00") (footprint "Inductor_SMD:L_0603_1608Metric")
     )
     (path "/5f304c88-142b-41d9-b86f-2d4158492d4d/9ed9ea2f-e5c2-42f9-bb2b-cbaec55eb2c9"
@@
     )
     (path "/5f304c88-142b-41d9-b86f-2d4158492d4d/c3e842d1-6265-4bbc-b262-9e817d5bb7a9"
-      (reference "U4") (unit 1) (value "93C46") (footprint "Package_SO:SO-8_3.9x4.9mm_P1.27mm")
+      (reference "U4") (unit 1) (value "93LC46B") (footprint "Package_SO:SO-8_3.9x4.9mm_P1.27mm")
     )
     (path "/5f304c88-142b-41d9-b86f-2d4158492d4d/32fbccdc-140b-45fb-8942-ec18d57e877b"
